File: Shield/Shield.kicad_sch (KiCad schematic)
At the start: 2 parts, among them U1 25aa040a-i/p, U2 ESP32-S3-DevKitC

Commit message: change address calling
Connections:
- net +5V: now also U1.7 (HOLD*)
- net HOLD: no longer names the net of U2.29 (GPIO48)
- net HOLD: no longer U1.7 (HOLD*)
- no-connect marks 32 -> 33
Changed lines of the file:
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@@
 		(company "BYU-I")
 	)
+	(junction
+		(at 195.58 45.72)
+		(diameter 0)
+		(color 0 0 0 0)
+	)
 	(no_connect
 		(at 93.98 71.12)
@@
 	)
 	(no_connect
+		(at 93.98 124.46)
+	)
+	(no_connect
 		(at 93.98 76.2)
 	)
@@
 	(wire
 		(pts
+			(xy 195.58 48.26) (xy 191.77 48.26)
+		)
+		(stroke
+			(width 0)
+			(type default)
+		)
+	)
+	(wire
+		(pts
+			(xy 195.58 45.72) (xy 195.58 48.26)
+		)
+		(stroke
+			(width 0)
+			(type default)
+		)
+	)
+	(wire
+		(pts
 			(xy 195.58 45.72) (xy 195.58 40.64)
 		)
@@
 		)
 	)
-	(global_label "HOLD"
-		(shape input)
-		(at 191.77 48.26 0)
-		(fields_autoplaced yes)
-		(effects
-			(font
-				(size 1.27 1.27)
-			)
-			(justify left)
-		)
-		(property "Intersheetrefs" "${INTERSHEET_REFS}"
-			(at 199.7143 48.26 0)
-			(effects
-				(font
-					(size 1.27 1.27)
-				)
-				(justify left)
-				(hide yes)
-			)
-		)
-	)
 	(global_label "SCK"
 		(shape input)
@@
 			(effects
 				(font
-					(size 1.27 1.27)
-				)
-				(justify left)
-				(hide yes)
-			)
-		)
-	)
-	(global_label "HOLD"
-		(shape input)
-		(at 93.98 124.46 0)
-		(fields_autoplaced yes)
-		(effects
-			(font
-				(size 1.27 1.27)
-			)
-			(justify left)
-		)
-		(property "Intersheetrefs" "${INTERSHEET_REFS}"
-			(at 101.9243 124.46 0)
-			(effects
-				(font

Commit message: Added level shifter
Parts:
- added Q1: BSS138, Package_TO_SOT_SMD:SOT-23, symbol Transistor_FET:BSS138
- added R1, R2: R_US, Resistor_SMD:R_0805_2012Metric_Pad1.20x1.40mm_HandSolder, symbol Device:R_US
Connections:
- net +5V: now also R1.1
- net +3V3: now reaches U2.1 (3V3), U2.2 (3V3)
- net +3V3: now also U2.29 (GPIO48), Q1.1 (G), R2.1
- net WP renamed HVWP
- net HVWP: now also Q1.3 (D), R1.2; no longer U2.20 (GPIO14/ADC2_CH3)
- new net LVWP: Q1.2 (S), R2.2, U2.20 (GPIO14/ADC2_CH3)
- no-connect marks 33 -> 31
Other:
- note added: "10K Ohm"
